File: hardware/BREAD_Slice.kicad_pcb (KiCad board)
At the start: 2 copper layers, 72.6 x 100 mm, 16 parts, among them J1 Conn_01x10_Female, J2 I2C_01x04

Commit message: Initial commit
Parts:
- removed C3, C4: 22uF, Capacitor_SMD:C_1206_3216Metric
- removed D1: WS2812B_5050, SparkFun-LED:WS2812-5050-4PIN
- removed HS1: Heatsink_Pad, SparkFun-Fuse:Thermal Pad
- removed L1: 4.7uH, Inductor_SMD:L_1210_3225Metric
- added J3: Term_2, OCI:TerminalBlock_Pheonix_MKDS1.5-2pol, F.Cu at (182.9, 85.2)
- added J4: Term_2, OCI:TerminalBlock_Pheonix_MKDS1.5-2pol, F.Cu at (182.9, 95.7)
- added Q1: TIP120, Package_TO_SOT_THT:TO-220-3_Vertical, F.Cu at (173.3, 85.2)
- added R1: 1k, OCI:R_1206_HandSoldering, B.Cu at (145.6, 63.6)
- added R2: 1k, OCI:R_1206_HandSoldering, B.Cu at (164.4, 63.6)
- added R3: 1k, OCI:R_1206_HandSoldering, B.Cu at (164.4, 71.0)
- added R4: 4k, OCI:R_1206_HandSoldering, B.Cu at (145.6, 71.0)
- C1: value 22uF -> 10uF_t; footprint Capacitor_SMD:C_1206_3216Metric -> OCI_UPL_FOOTPRINTS:C_2312
- C2: value 100nF -> 10uF_t; footprint Capacitor_SMD:C_1206_3216Metric -> OCI_UPL_FOOTPRINTS:C_2312
- H1, H4: footprint MountingHole:MountingHole_5mm -> MountingHole:MountingHole_3.2mm_M3_DIN965_Pad
- H2: renamed from H3; footprint MountingHole:MountingHole_5mm -> MountingHole:MountingHole_3.2mm_M3_DIN965_Pad
- H3: renamed from H2; footprint MountingHole:MountingHole_5mm -> MountingHole:MountingHole_3.2mm_M3_DIN965_Pad
- J2: value I2C_01x04 -> Term_2; footprint Connector_JST:JST_SH_SM04B-SRSS-TB_1x04-1MP_P1.00mm_Horizontal -> OCI:TerminalBlock_Pheonix_MKDS1.5-2pol; moved to F.Cu
- U1: value ~ -> LM358; footprint Package_TO_SOT_SMD:TSOT-23-6 -> OCI:DIP-8_W7.62mm_LongPads; moved to F.Cu
- moved Logo1 80.0 mm to (177.1, 134.3), turned to 0 degrees
- moved J2 69.8 mm to (182.9, 74.7), turned to 90 degrees
- moved U1 59.4 mm to (158.8, 71.5), turned to 180 degrees
- moved C1 34.1 mm to (154.6, 97.4), turned to 90 degrees
- moved C2 28.4 mm to (154.6, 110.2), turned to -90 degrees
- moved A1 7.59 mm to (135.0, 100.0)
- moved J1 3.43 mm to (129.6, 78.8)
Connections:
- A1 pad 19: unconnected-(A1-A0-Pad19) -> /A_TO_PUMP
- A1 pad 20: unconnected-(A1-A1-Pad20) -> /A_FB
- A1 pad 21: unconnected-(A1-A2-Pad21) -> /start_sw
- A1 pad 22: unconnected-(A1-A3-Pad22) -> /error_io
- A1 pad 30: unconnected-(A1-VIN-Pad30) -> +12V
- A1 pad 8: /LED -> unconnected-(A1-Pad8)
- C1 pad 1: GND -> +12V
- C1 pad 2: +12V -> GND
- C2 pad 1: Net-(U1-SW) -> +5V
- C2 pad 2: Net-(U1-BST) -> GND
- J2 pad 1: GND -> /A_IN
- J2 pad 2: +5V -> /A_OUT
- U1 pad 1: +5V -> /A_IN
- U1 pad 2: +12V -> Net-(R2-Pad2)
- U1 pad 3: +12V -> /A_TO_PUMP
- U1 pad 5: Net-(U1-SW) -> /A_OUT
- U1 pad 6: Net-(U1-BST) -> Net-(R1-Pad2)
Routing:
- net +5V: track 108.9 -> 4.37 mm, vias 1 -> 0
- net /A_TO_PUMP: track 0.00 -> 69.4 mm
- net /A_FB: track 0.00 -> 61.8 mm
- net /start_sw: track 0.00 -> 55.3 mm, vias 0 -> 1
- net /LED: track 51.5 -> 0.00 mm
- net /error_io: track 0.00 -> 45.3 mm
- net /A_OUT: track 0.00 -> 40.3 mm
- net /I2C_CLK: track 78.5 -> 40.0 mm, vias 2 -> 1
- net /I2C_DAT: track 76.6 -> 41.7 mm, vias 2 -> 1
- net +12V: track 46.8 -> 79.7 mm
- net /A_IN: track 0.00 -> 25.4 mm
- net /start: track 0.00 -> 10.7 mm
- net Net-(R1-Pad2): track 0.00 -> 9.28 mm
- net Net-(R2-Pad2): track 0.00 -> 8.97 mm
- net /E_STOP: track 30.1 -> 22.4 mm
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Other:
- board size 72.6 x 100 mm -> 70 x 100 mm
- board text added: "AIN |"
- board text added: "AOUT |"
- board text added: "GND |"
- board text added: "Pump Control Slice SLC_PUMP R0 2022"
- board text added: "START |"
- board text added: "| ERR |"
- board text removed: "12V"
- board text removed: "12V->5V Reg"
- board text removed: "5V I2C Connector"
- board text removed: "ARDUINO NANO"
- board text removed: "BREAD Slice Template SLC_TEMP <version> <year>"
- board text removed: "ESTOP"
- board text removed: "GND"
- board text removed: "INT"
- board text removed: "LED"
- board text removed: "SCL"
- board text removed: "SDA"
- board text removed: "SYNC"
