File: hardware/BREAD_Slice.kicad_sch (KiCad schematic)
At the start: 15 parts, among them J1 Conn_01x10_Female, J2 I2C_01x04

Commit message: Initial commit
Parts:
- removed C1, C3, C4: 22uF, Capacitor_SMD:C_1206_3216Metric, symbol Device:C_Small
- removed C2: 100nF, Capacitor_SMD:C_1206_3216Metric, symbol Device:C_Small
- removed D1: WS2812B_5050, SparkFun-LED:WS2812-5050-4PIN, symbol SparkFun-LED:WS2812B_5050
- removed HS1: Heatsink_Pad, SparkFun-Fuse:Thermal Pad, symbol Mechanical:Heatsink_Pad
- removed J2: I2C_01x04, Connector_JST:JST_SH_SM04B-SRSS-TB_1x04-1MP_P1.00mm_Horizontal, symbol SparkFun-Connector:I2C_01x04
- removed L1: 4.7uH, Inductor_SMD:L_1210_3225Metric, symbol Device:L_Small
- removed U1: ~, Package_TO_SOT_SMD:TSOT-23-6, symbol SparkFun-DiscreteSemi:AP63205
- added C1, C2: 10uF_t, OCI_UPL_FOOTPRINTS:C_2312, symbol OCI_UPL_2_Capacitors:10uF_t
- added J2, J3, J4: Term_2, OCI:TerminalBlock_Pheonix_MKDS1.5-2pol, symbol OCI_UPL_10_Connectors:Term_2
- added Logo1: Logo_Open_Hardware_Small, Symbol:OSHW-Symbol_6.7x6mm_SilkScreen, symbol Graphic:Logo_Open_Hardware_Small
- added Q1: TIP120, Package_TO_SOT_THT:TO-220-3_Vertical, symbol Transistor_BJT:TIP120
- added R1, R2, R3: 1k, OCI:R_1206_HandSoldering, symbol Device:R_US
- added R4: 4k, OCI:R_1206_HandSoldering, symbol Device:R_US
- added U1: LM358, OCI:DIP-8_W7.62mm_LongPads, symbol Amplifier_Operational:LM358
- H1, H4: footprint MountingHole:MountingHole_5mm -> MountingHole:MountingHole_3.2mm_M3_DIN965_Pad
- H2: renamed from H3; footprint MountingHole:MountingHole_5mm -> MountingHole:MountingHole_3.2mm_M3_DIN965_Pad
- H3: renamed from H2; footprint MountingHole:MountingHole_5mm -> MountingHole:MountingHole_3.2mm_M3_DIN965_Pad
Connections:
- net +12V: now also A1.30 (VIN), C1.1, U1.8 (V+)
- net +5V: now also C2.1
- net GND: now also C1.2, C2.2, J3.2, J4.2, Q1.3 (E), R1.1, R2.1, U1.4 (V-)
- net A_TO_PUMP: now reaches A1.19 (A0)
- net A_TO_PUMP: now also U1.3 (+)
- net A_FB: now reaches A1.20 (A1)
- net A_FB: now also R4.2, U1.7
- net start_sw: now reaches A1.21 (A2)
- net start_sw: now also Q1.1 (B)
- net error_io: now reaches A1.22 (A3)
- net error_io: now also J4.1
- net LED: no longer names the net of A1.8 (D5)
- new net: R2.2, R3.1, U1.2 (-)
- new net: R1.2, R4.1, U1.6 (-)
- new net A_IN: J2.1, R3.2, U1.1
- new net A_OUT: J2.2, U1.5 (+)
- new net start: J3.1, Q1.2 (C)
- no-connect marks 22 -> 17
Other:
- moved on the sheet: A1, H1, H2, H3, H4, J1
